File: KiCad files/Garden Control System/Sensors and HSDs.kicad_sch (KiCad schematic)
At the start: 23 parts, among them U3 UCC27624DR, U4 INA4180A2IPWR, U5 UCC27624DR, U6 IRLML6344TRPBF, U7 IRLML6344TRPBF, U8 IRLML6344TRPBF

Commit message: working on temp sensor circuit
Parts:
- added R40, R41: 220, symbol Device:R
- R24, R25, R26: value 221 -> 220
Connections:
- net at U5.1 (ENA), U5.8 (ENB): now also R41.2
- net at U3.1 (ENA), U3.8 (ENB): now also R40.2
- new net GDRIVER_EN: R40.1, R41.1
Other:
- note removed: "Supply 3.3V from buck and Vdd from Vin UCC21550BDWR"
- note removed: "Tie enable to pullup? 3v3? Micro Pin?"
Changed lines of the file:
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@@
 	)
 	(junction
+		(at 38.1 68.58)
+		(diameter 0)
+		(color 0 0 0 0)
+	)
+	(junction
 		(at 86.36 163.83)
 		(diameter 0)
@@
 	)
 	(junction
+		(at 38.1 124.46)
+		(diameter 0)
+		(color 0 0 0 0)
+	)
+	(junction
 		(at 119.38 149.86)
 		(diameter 0)
@@
 	(wire
 		(pts
-			(xy 35.56 81.28) (xy 39.37 81.28)
+			(xy 38.1 81.28) (xy 39.37 81.28)
 		)
 		(stroke
@@
 	(wire
 		(pts
+			(xy 24.13 68.58) (xy 27.94 68.58)
+		)
+		(stroke
+			(width 0)
+			(type default)
+		)
+	)
+	(wire
+		(pts
 			(xy 171.45 143.51) (xy 171.45 140.97)
 		)
@@
 	(wire
 		(pts
-			(xy 35.56 124.46) (xy 82.55 124.46)
+			(xy 38.1 124.46) (xy 82.55 124.46)
 		)
 		(stroke
@@
 	(wire
 		(pts
-			(xy 35.56 138.43) (xy 35.56 124.46)
+			(xy 38.1 138.43) (xy 38.1 124.46)
 		)
 		(stroke
@@
 	(wire
 		(pts
+			(xy 34.29 124.46) (xy 38.1 124.46)
+		)
+		(stroke
+			(width 0)
+			(type default)
+		)
+	)
+	(wire
+		(pts
 			(xy 218.44 137.16) (xy 218.44 146.05)
 		)
@@
 	(wire
 		(pts
-			(xy 35.56 68.58) (xy 35.56 81.28)
+			(xy 38.1 68.58) (xy 38.1 81.28)
 		)
 		(stroke
@@
 	(wire
 		(pts
-			(xy 81.28 68.58) (xy 35.56 68.58)
+			(xy 35.56 68.58) (xy 38.1 68.58)
+		)
+		(stroke
+			(width 0)
+			(type default)
+		)
+	)
+	(wire
+		(pts
+			(xy 81.28 68.58) (xy 38.1 68.58)
 		)
 		(stroke
@@
 	(wire
 		(pts
+			(xy 22.86 124.46) (xy 26.67 124.46)
+		)
+		(stroke
+			(width 0)
+			(type default)
+		)
+	)
+	(wire
+		(pts
 			(xy 39.37 86.36) (xy 38.1 86.36)
 		)
@@
 	(wire
 		(pts
-			(xy 40.64 138.43) (xy 35.56 138.43)
+			(xy 40.64 138.43) (xy 38.1 138.43)
 		)
 		(stroke
@@
 		)
 	)
-	(text_box "Current/Voltage monitoring ICs\nDigital with I2C:INA3221AIRGVR (3 CHANNEL) ~$6\nAnalog output: INA4180A2IPWR 4channel $1.5\nAnalog output: INA2180A1IDGKR 2channel $0.9\n\nFor analog option, might need to filter before micro..\nReview datasheet\n\nHigh side current sense above motor but below driver."
+	(text_box "Current/Voltage monitoring ICs\nDigital with I2C:INA3221AIRGVR (3 CHANNEL) ~$6\nAnalog output: INA4180A2IPWR 4channel $1.5\nAnalog output: INA2180A1IDGKR 2channel $0.9\n\nFor analog option, might need to filter before micro..\nReview datasheet\n\nHigh side current sense above motor."
 		(exclude_from_sim no)
-		(at 278.13 13.97 0)
+		(at 290.83 15.24 0)
 		(size 68.58 20.32)
 		(stroke
@@
 		)
 	)
-	(text_box "Motor driver connected as a HSD.\n18V max motor driver DRV8848PWPR: $3.50\n48V max motor driver DRV8434PPWPR: 6.06\n\nCould do a gate driver + mosfet for 12V and 24V operation.\nMosfet: 4x IRLML6344TRPBF, $0.519 + 2x UCC27624DR (or UCC27624QDRQ1) $2.15: TOT=~$6\n\nGate driver IN# good for 3V logic. Vdd safe for 5-26V."
+	(text_box "Motor driver connected as a HSD.\n18V max motor driver DRV8848PWPR: $3.50\n48V max motor driver DRV8434PPWPR: 6.06\n\nCould do a gate driver + mosfet for 12V and 24V operation.\nMosfet: 4x IRLML6344TRPBF, $0.519 + 2x UCC27624DR (or UCC27624QDRQ1) $2.15: TOT=~$6\n\nGate driver IN# good for 3V logic. Vdd safe for 4.5-26V."
 		(exclude_from_sim no)
 		(at 22.86 17.78 0)
-		(size 77.47 36.83)
+		(size 77.47 21.59)
 		(stroke
 			(width 0)
@@
 			(font
 				(size 1.27 1.27)
-				(color 255 0 0 1)
+				(color 0 0 132 1)
 			)
 			(justify left)
@@
 		)
 	)
-	(text "Tie enable to pullup? 3v3? Micro Pin?"
-		(exclude_from_sim no)
-		(at 15.24 66.548 0)
-		(effects
-			(font
-				(size 1.27 1.27)
-				(color 255 0 0 1)
-			)
-			(justify left)
-		)
-	)
 	(text "RDS(on) max @V GS = 4.5V, 29 mΩ\nRDS(on) max @V GS = 2.5V, 37 mΩ"
 		(exclude_from_sim no)
@@
 		)
 	)
-	(text "Supply 3.3V from buck and Vdd from Vin \nUCC21550BDWR\n"
-		(exclude_from_sim no)
-		(at 65.278 58.166 0)
-		(effects
-			(font
-				(size 1.27 1.27)
-				(color 255 0 0 1)
-			)
-			(justify left)
-		)
-	)
 	(text "ADD FLYBACK PROTECTION"
 		(exclude_from_sim no)
@@
 	(text "For the best high-speed circuit performance and to prevent noise problems because the device draws current\nfrom the VDD pin to bias all internal circuits, use two VDD bypass capacitors. Also, use surface mount, low\nESR capacitors. \n\nA 0.1-μF ceramic capacitor should be located less than 1 mm from the VDD to GND pins of\nthe gate-driver device. \n\nIn addition, a larger capacitor (≥1 μF) must be connected in parallel (also as close to the\ndriver IC as possible) to help deliver the high-current peaks required by the load. The parallel combination of\ncapacitors presents a low impedance characteristic for the expected current levels and switching frequencies in\nthe application."
 		(exclude_from_sim no)
-		(at -103.886 104.14 0)
+		(at -102.108 103.378 0)
 		(effects
 			(font
@@
 		)
 	)
+	(global_label "GDRIVER_EN"
+		(shape input)
+		(at 22.86 124.46 180)
+		(fields_autoplaced yes)
+		(effects
+			(font
+				(size 1.27 1.27)
+			)
+			(justify right)
+		)
+		(property "Intersheetrefs" "${INTERSHEET_REFS}"
+			(at 8.5053 124.46 0)
+			(effects
+				(font
+					(size 1.27 1.27)
+				)
+				(justify right)
+				(hide yes)
+			)
+		)
+	)
 	(global_label "I_SENSE2_-"
 		(shape input)
@@
 		)
 	)
+	(global_label "GDRIVER_EN"
+		(shape input)
+		(at 24.13 68.58 180)
+		(fields_autoplaced yes)
+		(effects
+			(font
+				(size 1.27 1.27)
+			)
+			(justify right)
+		)
+		(property "Intersheetrefs" "${INTERSHEET_REFS}"
+			(at 9.7753 68.58 0)
+			(effects
+				(font
+					(size 1.27 1.27)
+				)
+				(justify right)
+				(hide yes)
+			)
+		)
+	)
 	(global_label "I_SENSE2_+"
 		(shape input)
@@
 			)
 		)
-		(property "Value" "221"
+		(property "Value" "220"
 			(at 27.432 86.36 90)
 			(effects
@@
 			)
 		)
-		(property "Value" "221"
+		(property "Value" "220"
 			(at 27.432 138.684 90)
 			(effects
@@
 			)
 		)
-		(property "Value" "221"
+		(property "Value" "220"
 			(at 27.432 81.534 90)
 			(effects
@@
 	(symbol
 		(lib_id "Device:R")
+		(at 30.48 124.46 90)
+		(unit 1)
+		(exclude_from_sim no)
+		(in_bom yes)
+		(on_board yes)
+		(dnp no)
+		(property "Reference" "R41"
+			(at 31.242 122.174 90)
+			(effects
+				(font
+					(size 1.27 1.27)
+				)
+			)
+		)
+		(property "Value" "220"
+			(at 26.162 122.174 90)
+			(effects
+				(font
+					(size 1.27 1.27)
+				)
+			)
+		)
+		(property "Footprint" ""
+			(at 30.48 126.238 90)
+			(effects
+				(font
+					(size 1.27 1.27)
+				)
+				(hide yes)
+			)
+		)
+		(property "Datasheet" "~"
+			(at 30.48 124.46 0)
+			(effects
+				(font
+					(size 1.27 1.27)
+				)
+				(hide yes)
+			)
+		)
+		(property "Description" ""
+			(at 30.48 124.46 0)
+			(effects
+				(font
+					(size 1.27 1.27)
+				)
+				(hide yes)
+			)
+		)
+		(pin "1"
+		)
+		(pin "2"
+		)
+		(instances
+			(project "Garden Control System"
+				(path "/be495e14-3da3-4129-8396-1871cb6cba29/9f2dbd4f-9250-47a2-9054-c36b37ba7178"
+					(reference "R41")
+					(unit 1)
+				)
+			)
+		)
+	)
+	(symbol
+		(lib_id "Device:R")
 		(at 232.41 147.32 180)
 		(unit 1)
@@
 					(unit 1)
 				)
+			)
+		)
+	)
+	(symbol
+		(lib_id "Device:R")
+		(at 31.75 68.58 90)
+		(unit 1)
+		(exclude_from_sim no)
+		(in_bom yes)
+		(on_board yes)
+		(dnp no)
+		(property "Reference" "R40"
+			(at 32.512 66.294 90)
+			(effects
+				(font
+					(size 1.27 1.27)
+				)
+			)
+		)
+		(property "Value" "220"
+			(at 27.432 66.294 90)
+			(effects
+				(font
+					(size 1.27 1.27)
+				)
+			)
+		)
+		(property "Footprint" ""
+			(at 31.75 70.358 90)
+			(effects
+				(font
+					(size 1.27 1.27)
+				)
+				(hide yes)
+			)
+		)
+		(property "Datasheet" "~"
+			(at 31.75 68.58 0)
+			(effects
+				(font
+					(size 1.27 1.27)
+				)
+				(hide yes)
+			)
+		)
+		(property "Description" ""
+			(at 31.75 68.58 0)
+			(effects
+				(font
+					(size 1.27 1.27)
+				)
+				(hide yes)
+			)
+		)
+		(pin "1"
+		)
+		(pin "2"
+		)
+		(instances
+			(project "Garden Control System"
+				(path "/be495e14-3da3-4129-8396-1871cb6cba29/9f2dbd4f-9250-47a2-9054-c36b37ba7178"
+					(reference "R40")
+					(unit 1)
+				)

Commit message: saving changes
Parts:
- removed C44: 10u, symbol Device:C_Small
- removed C45: 100n, symbol Device:C_Small
- removed U5: UCC27624DR, SOIC_D0008A_TEX, symbol UCC27624DR:UCC27624DR
- added Q1: NPN, symbol Simulation_SPICE:NPN
- added Q2: PNP, symbol Simulation_SPICE:PNP
- added U5: IRLML6344TRPBF, IRLML6344TRPBF:SOT95P240X112-3N, symbol IRLML6344TRPBF:IRLML6344TRPBF
Connections:
- net 5V_BUCK: now also Q1.1 (C)
- net GND: now also Q2.3 (E)
- net NMOS2_GATE: now also Q1.3 (E), Q2.1 (C)
- net at R41.2: now also U5.3 (D)
- net at R26.2: now also U5.1 (G)
- new net: Q1.2 (B), Q2.2 (B)
- no-connect marks 2 -> 0
Other:
- note added: "MOSFET ACTS AS AN ENABLE (BIASING ISSUES? REMOVE?)"
- moved on the sheet: R26, R41
