File: KiCad files/Garden Control System/MCU.kicad_sch (KiCad schematic)
At the start: 27 parts, among them SW2 SW_SPDT, U1 STM32F207ZGTx, Y1 ECS-160-8-37-CWY-TR3

Commit message: Added a basic readme
Parts:
- C9: value 1u -> 4u7
Changed lines of the file:
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@@
 		(fields_autoplaced yes)
 		(property "Reference" "C9"
-			(at 281.94 67.3163 0)
+			(at 281.94 67.3162 0)
 			(effects
 				(font
@@
 			)
 		)
-		(property "Value" "1u"
-			(at 281.94 69.8563 0)
+		(property "Value" "4u7"
+			(at 281.94 69.8562 0)
 			(effects
 				(font
