File: KiCad files/Garden Control System/Encoder and Display.kicad_sch (KiCad schematic)
At the start: 10 parts, among them SW1 RotaryEncoder_Switch

Commit message: we cookin' again. Added LSD and start temp sense section.
Other:
- note added: "Display"
- note added: "Encoder and Button"
- note added: "LCD? TFT?"
Changed lines of the file:
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@@
+		)
+	)
+	(rectangle
+		(start 15.24 15.24)
+		(end 101.6 106.68)
+		(stroke
+			(width 0)
+			(type default)
+		)
+		(fill
+			(type none)
+		)
+	)
+	(rectangle
+		(start 106.68 15.24)
+		(end 279.4 157.48)
+		(stroke
+			(width 0)
+			(type default)
+		)
+		(fill
+			(type none)
+		)
+	)
+	(text "Encoder and Button"
+		(exclude_from_sim no)
+		(at 54.356 22.86 0)
+		(effects
+			(font
+				(size 3.81 3.81)
+				(thickness 0.508)
+				(bold yes)
+				(color 0 0 0 1)
+			)
 		)
 	)
 	(text "Encoder with switch:\nPEC11R-4115F-S0018\nButton is active high"
 		(exclude_from_sim no)
-		(at 51.054 18.288 0)
+		(at 28.956 35.56 0)
 		(effects
 			(font
@@
 			)
 		)
+	)
+	(text "LCD? TFT? "
+		(exclude_from_sim no)
+		(at 191.008 33.02 0)
+		(effects
+			(font
+				(size 1.27 1.27)
+				(color 255 0 0 1)
+			)
+			(justify left)
+		)
+	)
+	(text "Display"
+		(exclude_from_sim no)
+		(at 194.564 21.59 0)
+		(effects
+			(font
+				(size 3.81 3.81)
+				(thickness 0.508)
+				(bold yes)
+				(color 0 0 0 1)
+			)
+		)
