File: KiCad files/Garden Control System/_autosave-Temperature Sensors.kicad_sch (KiCad schematic)
At the start: 7 parts, among them J8 TB003-500-P06BE, U5 TLV9102IDGKR

Commit message: we cookin' again. Added LSD and start temp sense section.
Other:
- note added: "B value refers to the R/T slope for a specific temp range. output range should be 0.5-3.25V 3.25V = 3.3*R1/(R1+R2)"
- note added: "NTC B25/50 3950 100k Sensors"
- note removed: "NTC B25/50 3950 Sensors"
Changed lines of the file:
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@@
 		)
 	)
-	(text "NTC B25/50 3950 Sensors"
+	(text "B value refers to the R/T slope for a specific temp range.\n\noutput range should be 0.5-3.25V\n3.25V = 3.3*R1/(R1+R2)"
+		(exclude_from_sim no)
+		(at 77.978 102.616 0)
+		(effects
+			(font
+				(size 1.27 1.27)
+			)
+			(justify left)
+		)
+	)
+	(text "NTC B25/50 3950 100k Sensors"
 		(exclude_from_sim no)
 		(at 148.59 21.336 0)
